Commit message: Configure AprilTag rotation, size, and TCP offset

File: src/uarm_driver/swiftpro/urdf/pro_model.xacro (robot description, xacro)
@@ -210,14 +210,4 @@
 	<origin xyz= "0.15852 0 0" rpy = " 0 0 0" />
 </joint>
-    <link name="tcp_link">
-        <collision>
-            <origin xyz="0 0 0 " rpy="0 0 0" />
-        </collision>
-    </link>
-    <joint name="tcp_joint" type="fixed">
-        <origin xyz="0.06 0 -0.073" rpy="0 0 0" />
-        <parent link="Link8" />
-        <child link="tcp_link" />
-    </joint>
 <!--
 <link name="Link9">
